File: KiCad Files/Controller.kicad_sch (KiCad schematic)
At the start: 26 parts, among them U1 ProS3D, U2 LT, U3 RT

Commit message: Updated to current KiCad Design
Parts:
- C1: renamed from C4; footprint Capacitor_SMD:C_01005_0402Metric_Pad0.57x0.30mm_HandSolder -> Capacitor_SMD:C_0402_1005Metric_Pad0.74x0.62mm_HandSolder
- C2: renamed from C3; footprint Capacitor_SMD:C_01005_0402Metric_Pad0.57x0.30mm_HandSolder -> Capacitor_SMD:C_0402_1005Metric_Pad0.74x0.62mm_HandSolder
- C3: renamed from C5; footprint Capacitor_SMD:C_01005_0402Metric_Pad0.57x0.30mm_HandSolder -> Capacitor_SMD:C_0402_1005Metric_Pad0.74x0.62mm_HandSolder
- C4: renamed from C6; footprint Capacitor_SMD:C_01005_0402Metric_Pad0.57x0.30mm_HandSolder -> Capacitor_SMD:C_0402_1005Metric_Pad0.74x0.62mm_HandSolder
- C5: renamed from C7; footprint Capacitor_SMD:C_01005_0402Metric_Pad0.57x0.30mm_HandSolder -> Capacitor_SMD:C_0402_1005Metric_Pad0.74x0.62mm_HandSolder
- C6: renamed from C8; footprint Capacitor_SMD:C_01005_0402Metric_Pad0.57x0.30mm_HandSolder -> Capacitor_SMD:C_0402_1005Metric_Pad0.74x0.62mm_HandSolder
- C7: renamed from C9; footprint Capacitor_SMD:C_01005_0402Metric_Pad0.57x0.30mm_HandSolder -> Capacitor_SMD:C_0402_1005Metric_Pad0.74x0.62mm_HandSolder
- C8: renamed from C10; footprint Capacitor_SMD:C_01005_0402Metric_Pad0.57x0.30mm_HandSolder -> Capacitor_SMD:C_0402_1005Metric_Pad0.74x0.62mm_HandSolder
Connections:
- net JoyLeftX: now also U1.16 (IO13); no longer U1.17 (IO12)
- net JoyLeftY: now also U1.17 (IO12); no longer U1.16 (IO13)
Changed lines of the file:
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@@
 	(wire
 		(pts
-			(xy 322.58 91.44) (xy 309.88 91.44)
+			(xy 397.51 172.72) (xy 397.51 177.8)
 		)
 		(stroke
@@
 	(wire
 		(pts
-			(xy 397.51 172.72) (xy 397.51 177.8)
+			(xy 226.06 163.83) (xy 223.52 163.83)
 		)
 		(stroke
@@
 	(wire
 		(pts
-			(xy 226.06 163.83) (xy 223.52 163.83)
+			(xy 424.18 24.13) (xy 426.72 24.13)
 		)
 		(stroke
@@
 	(wire
 		(pts
-			(xy 424.18 24.13) (xy 426.72 24.13)
+			(xy 358.14 179.07) (xy 365.76 179.07)
 		)
 		(stroke
@@
 	(wire
 		(pts
-			(xy 358.14 179.07) (xy 365.76 179.07)
+			(xy 210.82 63.5) (xy 222.25 63.5)
 		)
 		(stroke
@@
 	(wire
 		(pts
-			(xy 210.82 63.5) (xy 222.25 63.5)
+			(xy 309.88 63.5) (xy 322.58 63.5)
 		)
 		(stroke
@@
 	(wire
 		(pts
-			(xy 309.88 63.5) (xy 322.58 63.5)
+			(xy 384.81 64.77) (xy 396.24 64.77)
 		)
 		(stroke
@@
 	(wire
 		(pts
-			(xy 384.81 64.77) (xy 396.24 64.77)
+			(xy 309.88 88.9) (xy 322.58 88.9)
 		)
 		(stroke
@@
 	(wire
 		(pts
-			(xy 309.88 88.9) (xy 322.58 88.9)
-		)
-		(stroke
-			(width 0)
-			(type default)
-		)
-	)
-	(wire
-		(pts
 			(xy 269.24 142.24) (xy 269.24 147.32)
 		)
@@
 	(wire
 		(pts
+			(xy 309.88 91.44) (xy 322.58 91.44)
+		)
+		(stroke
+			(width 0)
+			(type default)
+		)
+	)
+	(wire
+		(pts
 			(xy 223.52 196.85) (xy 223.52 195.58)
 		)
@@
 	)
 	(label "JoyLeftX"
-		(at 322.58 91.44 180)
+		(at 322.58 88.9 180)
 		(effects
 			(font
@@
 	)
 	(label "JoyLeftY"
-		(at 322.58 88.9 180)
+		(at 322.58 91.44 180)
 		(effects
 			(font
@@
 		(dnp no)
 		(fields_autoplaced yes)
-		(property "Reference" "C6"
+		(property "Reference" "C4"
 			(at 396.2463 27.94 90)
 			(show_name no)
@@
 			)
 		)
-		(property "Footprint" "Capacitor_SMD:C_01005_0402Metric_Pad0.57x0.30mm_HandSolder"
+		(property "Footprint" "Capacitor_SMD:C_0402_1005Metric_Pad0.74x0.62mm_HandSolder"
 			(at 396.24 34.29 0)
 			(hide yes)
@@
 			(project "Controller"
 				(path "/e42be9dc-66c8-439d-b9b0-22b04166f60b"
-					(reference "C6")
+					(reference "C4")
 					(unit 1)
 				)
@@
 		(dnp no)
 		(fields_autoplaced yes)
-		(property "Reference" "C10"
+		(property "Reference" "C8"
 			(at 462.2863 30.48 90)
 			(show_name no)
@@
 			)
 		)
-		(property "Footprint" "Capacitor_SMD:C_01005_0402Metric_Pad0.57x0.30mm_HandSolder"
+		(property "Footprint" "Capacitor_SMD:C_0402_1005Metric_Pad0.74x0.62mm_HandSolder"
 			(at 462.28 36.83 0)
 			(hide yes)
@@
 			(project "Controller"
 				(path "/e42be9dc-66c8-439d-b9b0-22b04166f60b"
-					(reference "C10")
+					(reference "C8")
 					(unit 1)
 				)
@@
 		(dnp no)
 		(fields_autoplaced yes)
-		(property "Reference" "C3"
+		(property "Reference" "C2"
 			(at 350.5263 27.94 90)
 			(show_name no)
@@
 			)
 		)
-		(property "Footprint" "Capacitor_SMD:C_01005_0402Metric_Pad0.57x0.30mm_HandSolder"
+		(property "Footprint" "Capacitor_SMD:C_0402_1005Metric_Pad0.74x0.62mm_HandSolder"
 			(at 350.52 34.29 0)
 			(hide yes)
@@
 			(project "Controller"
 				(path "/e42be9dc-66c8-439d-b9b0-22b04166f60b"
-					(reference "C3")
+					(reference "C2")
 					(unit 1)
 				)
@@
 		(dnp no)
 		(fields_autoplaced yes)
-		(property "Reference" "C8"
+		(property "Reference" "C6"
 			(at 429.2663 29.21 90)
 			(show_name no)
@@
 			)
 		)
-		(property "Footprint" "Capacitor_SMD:C_01005_0402Metric_Pad0.57x0.30mm_HandSolder"
+		(property "Footprint" "Capacitor_SMD:C_0402_1005Metric_Pad0.74x0.62mm_HandSolder"
 			(at 429.26 35.56 0)
 			(hide yes)
@@
 			(project "Controller"
 				(path "/e42be9dc-66c8-439d-b9b0-22b04166f60b"
-					(reference "C8")
+					(reference "C6")
 					(unit 1)
 				)
@@
 		(dnp no)
 		(fields_autoplaced yes)
-		(property "Reference" "C9"
+		(property "Reference" "C7"
 			(at 462.2863 17.78 90)
 			(show_name no)
@@
 			)
 		)
-		(property "Footprint" "Capacitor_SMD:C_01005_0402Metric_Pad0.57x0.30mm_HandSolder"
+		(property "Footprint" "Capacitor_SMD:C_0402_1005Metric_Pad0.74x0.62mm_HandSolder"
 			(at 462.28 24.13 0)
 			(hide yes)
@@
 			(project "Controller"
 				(path "/e42be9dc-66c8-439d-b9b0-22b04166f60b"
-					(reference "C9")
+					(reference "C7")
 					(unit 1)
 				)
@@
 		(dnp no)
 		(fields_autoplaced yes)
-		(property "Reference" "C7"
+		(property "Reference" "C5"
 			(at 429.2663 17.78 90)
 			(show_name no)
@@
 			)
 		)
-		(property "Footprint" "Capacitor_SMD:C_01005_0402Metric_Pad0.57x0.30mm_HandSolder"
+		(property "Footprint" "Capacitor_SMD:C_0402_1005Metric_Pad0.74x0.62mm_HandSolder"
 			(at 429.26 24.13 0)
 			(hide yes)
@@
 			(project "Controller"
 				(path "/e42be9dc-66c8-439d-b9b0-22b04166f60b"
-					(reference "C7")
+					(reference "C5")
 					(unit 1)
 				)
@@
 		(dnp no)
 		(fields_autoplaced yes)
-		(property "Reference" "C4"
+		(property "Reference" "C1"
 			(at 351.7963 17.78 90)
 			(show_name no)
@@
 			)
 		)
-		(property "Footprint" "Capacitor_SMD:C_01005_0402Metric_Pad0.57x0.30mm_HandSolder"
+		(property "Footprint" "Capacitor_SMD:C_0402_1005Metric_Pad0.74x0.62mm_HandSolder"
 			(at 351.79 24.13 0)
 			(hide yes)
@@
 			(project "Controller"
 				(path "/e42be9dc-66c8-439d-b9b0-22b04166f60b"
-					(reference "C4")
+					(reference "C1")
 					(unit 1)
 				)
@@
 		(dnp no)
 		(fields_autoplaced yes)
-		(property "Reference" "C5"
+		(property "Reference" "C3"
 			(at 396.2463 17.78 90)
 			(show_name no)
@@
 			)
 		)
-		(property "Footprint" "Capacitor_SMD:C_01005_0402Metric_Pad0.57x0.30mm_HandSolder"
+		(property "Footprint" "Capacitor_SMD:C_0402_1005Metric_Pad0.74x0.62mm_HandSolder"
 			(at 396.24 24.13 0)
 			(hide yes)
@@
 			(project "Controller"
 				(path "/e42be9dc-66c8-439d-b9b0-22b04166f60b"
-					(reference "C5")
+					(reference "C3")
 					(unit 1)
 				)
